File: mass_slit.brd (EAGLE design)
At the start: 37.8 x 35.5 mm, 24 parts, among them IC1 PIC18F1220P

Commit message: update
Parts:
- renumbered R5 to R6
Connections:
- net N$9: now also R6.1; no longer R6.2
- net VDD: now also R6.2; no longer R6.1
Routing:
- net N$15: track 27.6 -> 82.2 mm, vias 2 -> 0
- net N$6: track 54.0 -> 34.6 mm
- net N$13: track 30.2 -> 21.3 mm
- net VSS: track 102.2 -> 94.0 mm
- net N$16: track 66.2 -> 70.6 mm, vias 1 -> 0
- net N$5: track 37.2 -> 41.4 mm
- net N$1: track 55.7 -> 52.7 mm
- net N$9: track 40.3 -> 37.8 mm
- net VDD: track 61.7 -> 62.3 mm
- net N$12: track 48.2 -> 48.6 mm, vias 1 -> 0

Commit message: updates
Parts:
- added PAD11, PAD12, PAD13, PAD14, RESET: (no value), wirepad:1,6/0,9
- moved PAD9 2.84 mm to (30.5, 29.2)
- moved PAD10 2.54 mm to (30.5, 25.4)
- moved R4 2.54 mm to (12.7, 27.9)
- moved R3 2.54 mm to (7.62, 27.9)
- moved R6 1.80 mm to (26.7, 12.7)
- moved C3 1.80 mm to (30.5, 10.2)
- moved C4 1.27 mm to (7.62, 12.7)
- moved C5 1.27 mm to (19.1, 12.7)
- moved R2 1.27 mm to (12.7, 12.7)
- moved J2 1.27 mm to (15.2, 1.27)
- moved R1 1.27 mm to (30.5, 3.81)
- moved C1 1.27 mm to (31.8, 21.6)
- moved J1 1.27 mm to (15.2, 8.89)
- moved LED1 1.27 mm to (31.8, 16.5)
- renumbered PAD1 to P8, PAD2 to O-, PAD3 to O+, PAD4 to P5, PAD5 to P3, PAD6 to IN-, PAD7 to IN+
Connections:
- new net N$10: IC1.13, PAD12.1
- new net N$19: IC1.12, PAD11.1
- new net N$20: IC1.7, PAD13.1
- new net N$21: IC1.3, PAD14.1
- net N$7: now also RESET.1
Routing:
- net N$15: track 82.2 -> 33.3 mm
- net N$7: track 18.6 -> 52.3 mm
- net N$16: track 70.6 -> 37.5 mm
- net N$20: track 0.00 -> 23.0 mm
- net VDD: track 62.3 -> 85.3 mm
- net N$21: track 0.00 -> 20.2 mm
- net N$19: track 0.00 -> 19.1 mm
- net N$10: track 0.00 -> 11.9 mm
- net N$1: track 52.7 -> 62.3 mm
- net VSS: track 94.0 -> 86.6 mm
- net N$12: track 48.6 -> 54.4 mm
- net N$5: track 41.4 -> 47.0 mm
- net N$9: track 37.8 -> 32.6 mm, vias 0 -> 1
- net N$13: track 21.3 -> 26.1 mm
- net N$8: track 11.7 -> 14.4 mm
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Other:
- board size 37.8 x 35.5 mm -> 37.8 x 39.4 mm

Commit message: updates
Parts:
- added LED2: (no value), led:LED3MM
- added R5: (no value), resistor:0204V
- moved R3 8.89 mm to (16.5, 27.9), turned to 90 degrees
- moved R4 6.35 mm to (19.1, 27.9), turned to 90 degrees
- moved C6 3.81 mm to (24.1, 27.9)
- moved PAD8 2.54 mm to (27.9, 27.9)
Connections:
- new net N$22: IC1.6, R5.1
- new net N$23: LED2.K, R5.2
- net VDD: now also LED2.A
Routing:
- net VSS: track 86.6 -> 107.1 mm
- net N$20: track 23.0 -> 41.1 mm, vias 0 -> 1
- net N$7: track 52.3 -> 35.5 mm, vias 0 -> 1
- net N$9: track 32.6 -> 42.1 mm, vias 1 -> 0
- net N$8: track 14.4 -> 6.20 mm
- net N$12: track 54.4 -> 60.5 mm
- net N$13: track 26.1 -> 20.3 mm
- net N$23: track 0.00 -> 5.59 mm
- net N$1: track 62.3 -> 66.5 mm
- net N$5: track 47.0 -> 43.4 mm
- net N$19: track 19.1 -> 16.5 mm
- net N$22: track 0.00 -> 2.55 mm
- net N$6: track 37.2 -> 35.1 mm
- net N$4: track 17.1 -> 18.0 mm
- net N$2: track 14.6 -> 15.4 mm

Commit message: up
Parts:
- C1, C4, C6: value (none) -> 10uf
- C3, C5: value (none) -> 0.1
- R1: value (none) -> 2000
- R2, R4, R5: value (none) -> 220
- R3: value (none) -> 10000
- renumbered IN+ to IN-24, IN- to IN+24
Connections:
- net N$5 renamed -24
- net N$6 renamed +24
Changed lines of the file:
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@@
 <?xml version="1.0" encoding="utf-8"?>
 <!DOCTYPE eagle SYSTEM "eagle.dtd">
-<eagle version="9.2.2">
+<eagle version="9.4.1">
 <drawing>
 <settings>
@@
 <attribute name="VALUE" x="21.59" y="32.35" size="0.0254" layer="27"/>
 </element>
-<element name="IN-" library="wirepad" package="1,6/0,9" value="" x="24.13" y="31.75" smashed="yes">
+<element name="IN+24" library="wirepad" package="1,6/0,9" value="" x="24.13" y="31.75" smashed="yes">
 <attribute name="NAME" x="23.368" y="32.766" size="1.27" layer="25" ratio="10"/>
 <attribute name="VALUE" x="24.13" y="32.35" size="0.0254" layer="27"/>
 </element>
-<element name="IN+" library="wirepad" package="1,6/0,9" value="" x="26.67" y="31.75" smashed="yes">
+<element name="IN-24" library="wirepad" package="1,6/0,9" value="" x="26.67" y="31.75" smashed="yes">
 <attribute name="NAME" x="25.908" y="32.766" size="1.27" layer="25" ratio="10"/>
 <attribute name="VALUE" x="26.67" y="32.35" size="0.0254" layer="27"/>
 </element>
-<element name="C1" library="resistor" package="C025-040X050" value="" x="31.75" y="21.59" smashed="yes" rot="R270">
+<element name="C1" library="resistor" package="C025-040X050" value="10uf" x="31.75" y="21.59" smashed="yes" rot="R270">
 <attribute name="NAME" x="33.909" y="23.876" size="1.27" layer="25" ratio="10" rot="R270"/>
 <attribute name="VALUE" x="28.321" y="23.876" size="1.27" layer="27" ratio="10" rot="R270"/>
 </element>
-<element name="C3" library="capacitor-wima" package="C5B2.5" value="" x="30.48" y="10.16" smashed="yes">
+<element name="C3" library="capacitor-wima" package="C5B2.5" value="0.1" x="30.48" y="10.16" smashed="yes">
 <attribute name="NAME" x="28.448" y="11.684" size="1.27" layer="25" ratio="10"/>
 <attribute name="VALUE" x="28.448" y="7.366" size="1.27" layer="27" ratio="10"/>
 </element>
-<element name="C4" library="resistor" package="C025-040X050" value="" x="7.62" y="12.7" smashed="yes">
+<element name="C4" library="resistor" package="C025-040X050" value="10uf" x="7.62" y="12.7" smashed="yes">
 <attribute name="NAME" x="5.334" y="14.859" size="1.27" layer="25" ratio="10"/>
 <attribute name="VALUE" x="5.334" y="9.271" size="1.27" layer="27" ratio="10"/>
 </element>
-<element name="C5" library="capacitor-wima" package="C5B2.5" value="" x="19.05" y="12.7" smashed="yes">
+<element name="C5" library="capacitor-wima" package="C5B2.5" value="0.1" x="19.05" y="12.7" smashed="yes">
 <attribute name="NAME" x="17.018" y="14.224" size="1.27" layer="25" ratio="10"/>
 <attribute name="VALUE" x="17.018" y="9.906" size="1.27" layer="27" ratio="10"/>
 </element>
-<element name="C6" library="resistor" package="C025-040X050" value="" x="24.13" y="27.94" smashed="yes">
+<element name="C6" library="resistor" package="C025-040X050" value="10uf" x="24.13" y="27.94" smashed="yes">
 <attribute name="NAME" x="21.844" y="30.099" size="1.27" layer="25" ratio="10"/>
 <attribute name="VALUE" x="21.844" y="24.511" size="1.27" layer="27" ratio="10"/>
@@
 <attribute name="VALUE" x="5.1638" y="11.1407" size="1.27" layer="27"/>
 </element>
-<element name="R1" library="resistor" package="RTRIM3339P" value="" x="30.48" y="3.81" smashed="yes" rot="R180">
+<element name="R1" library="resistor" package="RTRIM3339P" value="2000" x="30.48" y="3.81" smashed="yes" rot="R180">
 <attribute name="NAME" x="32.995" y="-0.395" size="1.27" layer="25" rot="R180"/>
 <attribute name="VALUE" x="32.995" y="9.415" size="1.27" layer="27" rot="R180"/>
 </element>
-<element name="R2" library="resistor" package="0204V" value="" x="12.7" y="12.7" smashed="yes">
+<element name="R2" library="resistor" package="0204V" value="220" x="12.7" y="12.7" smashed="yes">
 <attribute name="NAME" x="10.5664" y="13.8684" size="1.27" layer="25" ratio="10"/>
 <attribute name="VALUE" x="10.5664" y="10.3886" size="1.27" layer="27" ratio="10"/>
 </element>
-<element name="R3" library="resistor" package="0204V" value="" x="16.51" y="27.94" smashed="yes" rot="R90">
+<element name="R3" library="resistor" package="0204V" value="10000" x="16.51" y="27.94" smashed="yes" rot="R90">
 <attribute name="NAME" x="15.3416" y="25.8064" size="1.27" layer="25" ratio="10" rot="R90"/>
 <attribute name="VALUE" x="18.8214" y="25.8064" size="1.27" layer="27" ratio="10" rot="R90"/>
 </element>
-<element name="R4" library="resistor" package="0204V" value="" x="19.05" y="27.94" smashed="yes" rot="R90">
+<element name="R4" library="resistor" package="0204V" value="220" x="19.05" y="27.94" smashed="yes" rot="R90">
 <attribute name="NAME" x="17.8816" y="25.8064" size="1.27" layer="25" ratio="10" rot="R90"/>
 <attribute name="VALUE" x="21.3614" y="25.8064" size="1.27" layer="27" ratio="10" rot="R90"/>
@@
 <attribute name="VALUE" x="30.48" y="33.62" size="0.0254" layer="27"/>
 </element>
-<element name="R5" library="resistor" package="0204V" value="" x="13.97" y="27.94" smashed="yes" rot="R90">
+<element name="R5" library="resistor" package="0204V" value="220" x="13.97" y="27.94" smashed="yes" rot="R90">
 <attribute name="NAME" x="12.8016" y="25.8064" size="1.27" layer="25" ratio="10" rot="R90"/>
 <attribute name="VALUE" x="16.2814" y="25.8064" size="1.27" layer="27" ratio="10" rot="R90"/>
@@
 <wire x1="31.9005" y1="20.196" x2="31.75" y2="20.32" width="0.254" layer="1"/>
 </signal>
-<signal name="N$5">
-<contactref element="IN+" pad="1"/>
+<signal name="-24">
+<contactref element="IN-24" pad="1"/>
 <contactref element="C4" pad="1"/>
 <contactref element="J1" pad="7"/>
@@
 <wire x1="6.426" y1="12.852" x2="6.35" y2="12.7" width="0.254" layer="16"/>
 </signal>
-<signal name="N$6">
-<contactref element="IN-" pad="1"/>
+<signal name="+24">
+<contactref element="IN+24" pad="1"/>
 <contactref element="C4" pad="2"/>
 <contactref element="J1" pad="8"/>

Commit message: up
Parts:
- R6: value (none) -> 330
Changed lines of the file:
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@@
 <?xml version="1.0" encoding="utf-8"?>
 <!DOCTYPE eagle SYSTEM "eagle.dtd">
-<eagle version="9.4.1">
+<eagle version="9.6.2">
 <drawing>
 <settings>
@@
 <attribute name="VALUE" x="5.1638" y="3.5207" size="1.27" layer="27"/>
 </element>
-<element name="R6" library="resistor" package="0204V" value="" x="26.67" y="12.7" smashed="yes">
+<element name="R6" library="resistor" package="0204V" value="330" x="26.67" y="12.7" smashed="yes">
 <attribute name="NAME" x="24.5364" y="13.8684" size="1.27" layer="25" ratio="10"/>
 <attribute name="VALUE" x="24.5364" y="10.3886" size="1.27" layer="27" ratio="10"/>
